File: ECS-Board/Rev A1/ABK-ECS - Rev A1.brd (EAGLE design)
At the start: 80 x 80 mm, 159 parts, among them J1 1241050-5, J2 USB-B-S-RA, J3 22-27-2061-06, J4 22-05-7068-06, J5 22-05-7028-02, J6 22-05-7028-02, J7 22-05-7068-06, K3 G6K-2G-Y, SW1 B3FS-1015, SW2 B3FS-1015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

Commit message: Update MPN and generate part list
Parts:
- C21: value 0.1Uf -> 0.1uF
Changed lines of the file:
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@@
 <grid distance="25" unitdist="mil" unit="mil" style="lines" multiple="2" display="yes" altdistance="12.5" altunitdist="mil" altunit="mil"/>
 <layers>
-<layer number="1" name="Top" color="16" fill="1" visible="no" active="yes"/>
-<layer number="2" name="Route2" color="17" fill="1" visible="no" active="yes"/>
+<layer number="1" name="Top" color="16" fill="1" visible="yes" active="yes"/>
+<layer number="2" name="Route2" color="17" fill="1" visible="yes" active="yes"/>
 <layer number="14" name="Route14" color="1" fill="6" visible="no" active="no"/>
-<layer number="15" name="Route15" color="19" fill="1" visible="no" active="yes"/>
+<layer number="15" name="Route15" color="19" fill="1" visible="yes" active="yes"/>
 <layer number="16" name="Bottom" color="21" fill="1" visible="yes" active="yes"/>
 <layer number="17" name="Pads" color="18" fill="1" visible="yes" active="yes"/>
@@
 <layer number="19" name="Unrouted" color="6" fill="1" visible="no" active="yes"/>
 <layer number="20" name="Dimension" color="7" fill="1" visible="yes" active="yes"/>
-<layer number="21" name="tPlace" color="55" fill="1" visible="no" active="yes"/>
+<layer number="21" name="tPlace" color="55" fill="1" visible="yes" active="yes"/>
 <layer number="22" name="bPlace" color="54" fill="1" visible="yes" active="yes"/>
-<layer number="23" name="tOrigins" color="15" fill="1" visible="no" active="yes"/>
+<layer number="23" name="tOrigins" color="15" fill="1" visible="yes" active="yes"/>
 <layer number="24" name="bOrigins" color="15" fill="1" visible="yes" active="yes"/>
-<layer number="25" name="tNames" color="55" fill="1" visible="no" active="yes"/>
+<layer number="25" name="tNames" color="55" fill="1" visible="yes" active="yes"/>
 <layer number="26" name="bNames" color="54" fill="1" visible="yes" active="yes"/>
-<layer number="27" name="tValues" color="53" fill="1" visible="no" active="yes"/>
+<layer number="27" name="tValues" color="53" fill="1" visible="yes" active="yes"/>
 <layer number="28" name="bValues" color="52" fill="1" visible="yes" active="yes"/>
 <layer number="29" name="tStop" color="7" fill="3" visible="no" active="yes"/>
@@
 <layer number="49" name="Reference" color="48" fill="1" visible="yes" active="yes"/>
 <layer number="50" name="dxf" color="7" fill="1" visible="yes" active="yes"/>
-<layer number="51" name="tDocu" color="55" fill="1" visible="no" active="yes"/>
+<layer number="51" name="tDocu" color="55" fill="1" visible="yes" active="yes"/>
 <layer number="52" name="bDocu" color="54" fill="1" visible="yes" active="yes"/>
 <layer number="53" name="tGND_GNDA" color="7" fill="1" visible="yes" active="yes"/>
@@
 <attribute name="OC_FARNELL" value="unknown" x="74.93" y="26.67" size="1.778" layer="27" rot="R90" display="off"/>
 <attribute name="MF" value="" x="74.93" y="26.67" size="1.778" layer="27" rot="R90" display="off"/>
-<attribute name="OC_NEWARK" value="25M1733" x="74.93" y="26.67" size="1.778" layer="27" rot="R90" display="off"/>
+<attribute name="OC_NEWARK" value="89K0316" x="74.93" y="26.67" size="1.778" layer="27" rot="R90" display="off"/>
 <attribute name="NAME" x="75.7824" y="35.1521" size="0.6096" layer="25" ratio="10"/>
 <attribute name="VALUE" x="75.7824" y="34.5171" size="0.4064" layer="27" ratio="10"/>
@@
 <attribute name="OC_FARNELL" value="unknown" x="74.93" y="52.07" size="1.778" layer="27" rot="R90" display="off"/>
 <attribute name="MF" value="" x="74.93" y="52.07" size="1.778" layer="27" rot="R90" display="off"/>
-<attribute name="OC_NEWARK" value="25M1733" x="74.93" y="52.07" size="1.778" layer="27" rot="R90" display="off"/>
+<attribute name="OC_NEWARK" value="89K0316" x="74.93" y="52.07" size="1.778" layer="27" rot="R90" display="off"/>
 <attribute name="NAME" x="75.4649" y="61.1871" size="0.6096" layer="25" ratio="10"/>
 <attribute name="VALUE" x="75.4649" y="60.2346" size="0.4064" layer="27" ratio="10"/>
@@
 <attribute name="VALUE" x="58.42" y="57.785" size="0.4064" layer="28" rot="MR0"/>
 </element>
-<element name="C21" library="rcl" package="C0603" value="0.1Uf" x="50.8" y="46.0375" smashed="yes" rot="R180">
-<attribute name="OC_NEWARK" value="06R4927" x="50.8" y="46.0375" size="1.778" layer="27" rot="R180" display="off"/>
+<element name="C21" library="rcl" package="C0603" value="0.1uF" x="50.8" y="46.0375" smashed="yes" rot="R180">
+<attribute name="OC_NEWARK" value="06R4923" x="50.8" y="46.0375" size="1.778" layer="27" rot="R180" display="off"/>
 <attribute name="MF" value="" x="50.8" y="46.0375" size="1.778" layer="27" rot="R180" display="off"/>
-<attribute name="MPN" value="MC0603B104K500CT" x="50.8" y="46.0375" size="1.778" layer="27" rot="R180" display="off"/>
+<attribute name="MPN" value="MC0603B104K160CT" x="50.8" y="46.0375" size="1.778" layer="27" rot="R180" display="off"/>
 <attribute name="NAME" x="49.2125" y="44.7675" size="0.6096" layer="25"/>
 <attribute name="VALUE" x="51.1175" y="44.7675" size="0.4064" layer="27"/>
@@
 <attribute name="NAME" x="3.4952" y="38.1" size="0.6096" layer="26" rot="MR180"/>
 <attribute name="VALUE" x="3.4952" y="41.021" size="0.4064" layer="28" rot="MR180"/>
+<attribute name="OC_NEWARK" value="unknown" x="4.445" y="39.37" size="1.778" layer="28" rot="MR180" display="off"/>
+<attribute name="MF" value="" x="4.445" y="39.37" size="1.778" layer="28" rot="MR180" display="off"/>
+<attribute name="MPN" value="" x="4.445" y="39.37" size="1.778" layer="28" rot="MR180" display="off"/>
 </element>
 </elements>
