File: ECS-Board/Rev A1/ABK-ECS - Rev A1.sch (EAGLE design)
At the start: 159 parts, among them J1 1241050-5, J2 USB-B-S-RA, J3 22-27-2061-06, J4 22-05-7068-06, J5 22-05-7028-02, J6 22-05-7028-02, J7 22-05-7068-06, K3 G6K-2G-Y, SW1 B3FS-1015, SW2 B3FS-1015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

Commit message: Update MPN and generate part list
Parts:
- C21: value 0.1Uf -> 0.1uF; MPN MC0603B104K500CT -> MC0603B104K160CT; OC_NEWARK 06R4927 -> 06R4923
- J4, J7: OC_NEWARK 25M1733 -> 89K0316
- SJ3: OC_NEWARK (none) -> unknown
Changed lines of the file:
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@@
 <part name="J4" library="con-molex" deviceset="22-?-06" device="05-7068">
 <attribute name="MPN" value="22-05-7068"/>
-<attribute name="OC_NEWARK" value="25M1733"/>
+<attribute name="OC_NEWARK" value="89K0316"/>
 </part>
 <part name="P+6" library="supply3" deviceset="+24V" device=""/>
@@
 <part name="J7" library="con-molex" deviceset="22-?-06" device="05-7068">
 <attribute name="MPN" value="22-05-7068"/>
-<attribute name="OC_NEWARK" value="25M1733"/>
+<attribute name="OC_NEWARK" value="89K0316"/>
 </part>
 <part name="P+18" library="supply3" deviceset="+24V" device=""/>
@@
 <part name="GND68" library="supply1" deviceset="GND" device=""/>
 <part name="+3V4" library="supply1" deviceset="+3V3" device=""/>
-<part name="C21" library="rcl" deviceset="C-EU" device="C0603" value="0.1Uf">
-<attribute name="MF" value=""/>
-<attribute name="MPN" value="MC0603B104K500CT"/>
-<attribute name="OC_NEWARK" value="06R4927"/>
+<part name="C21" library="rcl" deviceset="C-EU" device="C0603" value="0.1uF">
+<attribute name="MF" value=""/>
+<attribute name="MPN" value="MC0603B104K160CT"/>
+<attribute name="OC_NEWARK" value="06R4923"/>
 </part>
 <part name="+3V5" library="supply1" deviceset="+3V3" device=""/>
@@
 </part>
 <part name="GND8" library="supply1" deviceset="GND" device=""/>
-<part name="SJ3" library="SparkFun-Passives" deviceset="SOLDERJUMPER" device="NC"/>
+<part name="SJ3" library="SparkFun-Passives" deviceset="SOLDERJUMPER" device="NC">
+<attribute name="MF" value=""/>
+<attribute name="MPN" value=""/>
+<attribute name="OC_NEWARK" value="unknown"/>
+</part>
 <part name="GND78" library="supply1" deviceset="GND" device=""/>
 </parts>
@@
 <attribute name="MPN" x="24.13" y="17.78" size="1.778" layer="96" rot="R180" display="off"/>
 </instance>
-<instance part="SJ3" gate="1" x="187.96" y="30.48" rot="R90"/>
+<instance part="SJ3" gate="1" x="187.96" y="30.48" rot="R90">
+<attribute name="OC_NEWARK" x="187.96" y="30.48" size="1.778" layer="96" display="off"/>
+<attribute name="MF" x="187.96" y="30.48" size="1.778" layer="96" display="off"/>
+<attribute name="MPN" x="187.96" y="30.48" size="1.778" layer="96" display="off"/>
+</instance>
 <instance part="GND78" gate="1" x="187.96" y="20.32"/>
 </instances>
