File: ECS-Board/Rev A2/ABK-ECS - Rev A2.sch (EAGLE design)
At the start: 246 parts, among them J1 22-27-2061-06, J10 22-05-7068-06, J2 USB-B-S-RA, J3 1241050-5, J4 MSTBA2, J5 22-05-7068-06, J6 22-05-7028-02, J7 22-05-7068-06, J8 22-05-7068-06, J9 22-05-7028-02, K1 G6K-2G-Y, SW1 B3FS-1015, SW2 B3FS-1015, T1 EXMACHINA-LOGO-NAME, T10 MMBT2222AL, T11 MMBT2222AL, T12 IRLML5103TRPBF, T13 IRLML5103TRPBF, T14 IRLML5103TRPBF, T15 IRLML5103TRPBF, T16 MMBT2222AL, T17 MMBT2222AL, T18 MMBT2222AL, T19 MMBT2222AL, T2 IRLML5103TRPBF, T3 MMBT2222AL, T4 IRLML5103TRPBF, T5 IRLML5103TRPBF, T6 IRLML5103TRPBF, T7 IRLML5103TRPBF, T8 MMBT2222AL, T9 MMBT2222AL, U1 AT24C512C-SSHM-B, U2 LPC1768FBD100, U3 LT3686HDDPBF, U4 LT3686HDDPBF, U5 TC1264-3.3, U6 CD4050BD, U7 CD4050BD, X1 FC-135, X2 ASE-12, X3 3000

Commit message: Generate Gerber and MDP files
Parts:
- C10, C5: MPN MC0603N180K500CT -> GRM1885C1H180JA01D; OC_NEWARK 06R5140 -> 14T3328
- C14, C15: MPN MC0603B102K500CT -> GRM188R71H102KA01D; OC_NEWARK 06R4910 -> 19X1713
- C18, C19: MF (none) -> KEMET; MPN MCMT21N220F250CT -> C0805C226M9PACTU; OC_NEWARK 23T7233 -> 70K9142
- C20, C21: MPN (none) -> GRM188R61C105KA93D; OC_NEWARK (none) -> 03AC2661
- D10, D11, D12, D13, D14, D6, D7, D8, D9: MPN (none) -> 1N4148WS; OC_NEWARK (none) -> 31Y5518
- J10, J5, J8: MPN 22-05-7068 -> (none); OC_NEWARK 89K0316 -> (none)
- LED21: value 01.1 -> Blue
- LED5, LED6: device led:LEDCHIP-LED0603 -> led:LEDCHIPLED_0603
- OK2: MF (none) -> VISHAY/TELEFUNKEN; MPN (none) -> TCMT4100; OC_NEWARK (none) -> 06H1639
- R1: value 4K7 -> 4K7, DNI; MPN MCMR06X4701FTL -> RC0603FR-074K7L; OC_NEWARK 86T3649 -> 68R0092
- R10: value 0R -> 10K; MPN MCMR06X000 PTL -> RC0603FR-0710KL; OC_NEWARK 86T3500 -> 68R0049
- R100, R70, R71, R72, R98, R99: MPN MCMR06X4701FTL -> RC0603FR-07330RL; OC_NEWARK 86T3649 -> 98K7391
- R101, R64, R73: value 100 -> 330; MPN MCMR06X1000FTL -> RC0603FR-07330RL; OC_NEWARK 86T3504 -> 98K7391
- R102, R103, R104, R74, R75, R76: MPN MCMR06X1000FTL -> RC0603FR-13100RL; OC_NEWARK 86T3504 -> 68R0131
- R105, R40, R77: value 1K5 -> 100; MPN MCMR06X1501FTL -> RC0603FR-13100RL; OC_NEWARK 86T3542 -> 68R0131
- R106, R107, R108, R14, R24, R54, R55, R56, R57, R58, R59, R60, R61, R78, R79, R80: MPN MCMR06X1501FTL -> RC0603FR-071K5L; OC_NEWARK 86T3542 -> 68R0045
- R109, R81: value 4K7 -> 1K5; MPN MCMR06X4701FTL -> RC0603FR-071K5L; OC_NEWARK 86T3649 -> 68R0045
- R11: MPN MCMR06X000 PTL -> RC0603FR-070RL; OC_NEWARK 86T3500 -> 50Y7761
- R110, R111, R112, R18, R2, R3, R35, R36, R37, R38, R4, R50, R51, R52, R82, R83, R84: MPN MCMR06X4701FTL -> RC0603FR-074K7L; OC_NEWARK 86T3649 -> 68R0092
- R113, R85: value 1K -> 4K7; MPN MCMR06X1001FTL -> RC0603FR-074K7L; OC_NEWARK 86T3505 -> 68R0092
- R114, R115, R116, R27, R28, R29, R30, R31, R32, R33, R42, R43, R44, R45, R46, R47, R48, R86, R87, R88: MPN MCMR06X1001FTL -> RC0603FR-071KL; OC_NEWARK 86T3505 -> 68R0042
- R117, R89: value 330 -> 1K; MPN MCMR06X3300FTL -> RC0603FR-071KL; OC_NEWARK 86T3616 -> 68R0042
- R118, R119, R120, R90, R91, R92: MPN MCMR06X3300FTL -> RC0603FR-07330RL; OC_NEWARK 86T3616 -> 98K7391
- R12: value 10K -> 0R; MPN MCMR06X1002FTL -> RC0603FR-070RL; OC_NEWARK 86T3506 -> 50Y7761
- R121: value 0R -> 330; MPN MCMR06X000 PTL -> RC0603FR-07330RL; OC_NEWARK 86T3500 -> 98K7391
- R13, R23: value 1K5 -> 10K; MPN MCMR06X1501FTL -> RC0603FR-0710KL; OC_NEWARK 86T3542 -> 68R0049
- R15: value 31K6 -> 1K5; MPN MCMR06X3162FTL -> RC0603FR-071K5L; OC_FARNELL 2073391 -> (none); OC_NEWARK 86T3613 -> 68R0045
- R17: value 4K7 -> 31K6; MPN MCMR06X4701FTL -> MCMR06X3162FTL; OC_FARNELL (none) -> 2073391; OC_NEWARK 86T3649 -> 86T3613
- R19: value 52K3 -> 4K7; MPN MC0063W0603152K3 -> RC0603FR-074K7L; OC_FARNELL 2073391 -> (none); OC_NEWARK 26M0962 -> 68R0092
- R20: value 10K -> 52K3; MPN MCMR06X1002FTL -> MC0063W0603152K3; OC_NEWARK 86T3506 -> 26M0962
- R21: value 31K6 -> 10K; MPN MCMR06X3162FTL -> RC0603FR-0710KL; OC_NEWARK 86T3613 -> 68R0049
- R22: value 10K -> 31K6; MPN MCMR06X1002FTL -> MCMR06X3162FTL; OC_NEWARK 86T3506 -> 86T3613
- R25: value 100 -> 1K5; MPN MCMR06X1000FTL -> RC0603FR-071K5L; OC_FARNELL (none) -> 2073391; OC_NEWARK 86T3504 -> 68R0045
- R26: value 1K -> 100; MPN MCMR06X1001FTL -> RC0603FR-13100RL; OC_NEWARK 86T3505 -> 68R0131
- R34, R49: value 4K7 -> 1K; MPN MCMR06X4701FTL -> RC0603FR-071KL; OC_NEWARK 86T3649 -> 68R0042
- R39: value 100 -> 4K7; MPN MCMR06X1000FTL -> RC0603FR-074K7L; OC_NEWARK 86T3504 -> 68R0092
- R41: value 1K -> 1K5; MPN MCMR06X1001FTL -> RC0603FR-071K5L; OC_NEWARK 86T3505 -> 68R0045
- R5: value 33 -> 0R; MPN MCMR06X33R0FTL -> RC0603FR-070RL; OC_NEWARK 86T3614 -> 50Y7761
- R53: value 1K5 -> 4K7; MPN MCMR06X1501FTL -> RC0603FR-074K7L; OC_NEWARK 86T3542 -> 68R0092
- R6: MPN MCMR06X33R0FTL -> RC0603FR-0733RL; OC_NEWARK 86T3614 -> 68R0085
- R62: value 10K -> 1K5; MPN MCMR06X4701FTL -> RC0603FR-071K5L; OC_NEWARK 86T3649 -> 68R0045
- R63, R69, R97: value 330 -> 10K; MPN MCMR06X4701FTL -> RC0603FR-0710KL; OC_NEWARK 86T3649 -> 68R0049
- R65: value 10K -> 100; MPN MCMR06X4701FTL -> RC0603FR-13100RL; OC_NEWARK 86T3649 -> 68R0131
- R66, R67, R68, R94, R95, R96: MPN MCMR06X4701FTL -> RC0603FR-0710KL; OC_NEWARK 86T3649 -> 68R0049
- R7: value 1K5 -> 33; MPN MCMR06X1501FTL -> RC0603FR-0733RL; OC_NEWARK 86T3542 -> 68R0085
- R8: value 1K5 -> 1K5, DNI; MPN MCMR06X1501FTL -> RC0603FR-071K5L; OC_NEWARK 86T3542 -> 68R0045
- R9: value 10K -> 1K5, DNI; MPN MCMR06X1002FTL -> RC0603FR-071K5L; OC_NEWARK 86T3506 -> 68R0045
- R93: value 10K -> 330; MPN MCMR06X4701FTL -> RC0603FR-07330RL; OC_NEWARK 86T3649 -> 98K7391
- T10, T11, T16, T17, T18, T19, T3, T8, T9: MF (none) -> ON SEMICONDUCTOR; MPN (none) -> MMBT2222ALT1G; OC_NEWARK (none) -> 84K8795
- T12, T13, T14, T15, T2, T4, T5, T6, T7: MF (none) -> INTERNATIONAL RECTIFIER(IR); MPN (none) -> IRLML5103TRPBF; OC_NEWARK (none) -> 63J7612
- U1: MPN (none) -> AT24C512C-SSHM-B; OC_NEWARK (none) -> 68T4128
- U5: OC_NEWARK (none) -> unknown
Connections:
- net !RESET: now also R13.1; no longer R12.1
- net +24V: now also R101.2, R19.2, R64.2, R73.2; no longer R17.2, R63.2, R69.2, R97.2
- net +3V3: now also R10.2, R13.2, R22.2, R25.2, R9.1; no longer R12.2, R21.2, R24.2, R7.1, R9.2
- net +5V: now also R20.2, R24.2, R39.1, R41.2; no longer R19.2, R23.2, R38.1, R40.2
- net BOOT_SELECT_P2_10: now also R11.1, R5.1; no longer R10.1, R121.1
- net BOOT_SELECT_P2_12: now also R12.1; no longer R11.1
- net GND: now also R113.2, R15.2, R17.1, R21.1, R23.1, R38.2, R62.2, R63.1, R69.1, R85.2, R97.1; no longer R105.2, R13.2, R15.1, R20.1, R22.1, R34.2, R49.2, R62.1, R65.1, R77.2, R93.1
- net INPUT1.1: now also R49.2, R53.1; no longer R48.2, R52.1
- net INPUT1.2: now also R48.2, R52.1; no longer R47.2, R51.1
- net INPUT1.3: now also R47.2, R51.1; no longer R46.2, R50.1
- net INPUT1.4: now also R46.2, R50.1; no longer R45.2, R49.1
- net INPUT2.1: now also R34.2, R38.1; no longer R33.2, R37.1
- net INPUT2.2: now also R33.2, R37.1; no longer R32.2, R36.1
- net INPUT2.3: now also R32.2, R36.1; no longer R31.2, R35.1
- net INPUT2.4: now also R31.2, R35.1; no longer R30.2, R34.1
- net INPUT3.1: now also R40.2; no longer R39.2
- net ISP_RTS: now also R5.2; no longer R121.2
- net MOTOR_VFQ: now also R63.2; no longer R62.2
- net N$1: now also R7.1, R9.2; no longer R6.1, R8.2
- net N$100: now also R46.1; no longer R45.1
- net N$101: now also R43.2; no longer R42.2
- net N$102: now also R43.1; no longer R42.1
- net N$103: now also R47.1; no longer R46.1
- net N$104: now also R44.2; no longer R43.2
- net N$105: now also R44.1; no longer R43.1
- net N$106: now also R48.1; no longer R47.1
- net N$107: now also R59.1; no longer R58.1
- net N$108: now also R60.1; no longer R59.1
- net N$109: now also R61.1; no longer R60.1
- net N$110: now also R49.1; no longer R48.1
- net N$111: now also R45.2; no longer R44.2
- net N$112: now also R45.1; no longer R44.1
- net N$13: now also R22.1, R23.2; no longer R21.1, R22.2
- net N$17: now also R74.2; no longer R73.2
- net N$18: now also R70.1; no longer R69.1
- net N$19: now also R75.2; no longer R74.2
- net N$2: now also R6.1, R8.2; no longer R5.1, R7.2
- net N$20: now also R71.1; no longer R70.1
- net N$21: now also R76.2; no longer R75.2
- net N$22: now also R72.1; no longer R71.1
- net N$23: now also R77.2; no longer R76.2
- net N$24: now also R73.1; no longer R72.1
- net N$25: now also R65.1; no longer R64.1
- net N$26: now also R64.1; no longer R63.1
- net N$28: now also R26.2; no longer R25.2
- net N$29: now also R14.1; no longer R13.1
- net N$3: now also R15.1; no longer R14.1
- net N$31: now also R102.1, R110.1, R114.1; no longer R101.1, R109.1, R113.1
- net N$32: now also R26.1; no longer R25.1
- net N$33: now also R114.2; no longer R113.2
- net N$34: now also R103.1, R111.1, R115.1; no longer R102.1, R110.1, R114.1
- net N$35: now also R115.2; no longer R114.2
- net N$36: now also R104.1, R112.1, R116.1; no longer R103.1, R111.1, R115.1
- net N$37: now also R105.1, R113.1, R117.1; no longer R104.1, R112.1, R116.1
- net N$38: now also R116.2; no longer R115.2
- net N$39: now also R117.2; no longer R116.2
- net N$4: now also R16.2; no longer R15.2
- net N$40: now also R118.1; no longer R117.1
- net N$41: now also R27.2; no longer R26.2
- net N$42: now also R119.1; no longer R118.1
- net N$43: now also R121.1; no longer R120.1
- net N$44: now also R19.1; no longer R18.1
- net N$45: now also R18.1; no longer R17.1
- net N$46: now also R120.1; no longer R119.1
- net N$47: now also R28.2; no longer R27.2
- net N$48: now also R29.2; no longer R28.2
- net N$49: now also R30.2; no longer R29.2
- net N$5: now also R10.1, R12.2; no longer R10.2, R9.1
- net N$50: now also R25.1; no longer R24.1
- net N$51: now also R24.1; no longer R23.1
- net N$52: now also R30.1; no longer R29.1
- net N$53: now also R29.1; no longer R28.1
- net N$54: now also R28.1; no longer R27.1
- net N$55: now also R27.1; no longer R26.1
- net N$56: now also R54.1; no longer R53.1
- net N$57: now also R55.1; no longer R54.1
- net N$58: now also R56.1; no longer R55.1
- net N$59: now also R57.1; no longer R56.1
- net N$61: now also R34.1; no longer R33.1
- net N$62: now also R33.1; no longer R32.1
- net N$63: now also R32.1; no longer R31.1
- net N$64: now also R31.1; no longer R30.1
- net N$65: now also R58.1; no longer R57.1
- net N$66: now also R106.1; no longer R105.1
- net N$67: now also R107.1; no longer R106.1
- net N$68: now also R108.1; no longer R107.1
- net N$69: now also R109.1; no longer R108.1
- net N$7: now also R17.2; no longer R16.2
- net N$71: now also R98.1; no longer R97.1
- net N$72: now also R99.1; no longer R98.1
- net N$73: now also R39.2, R40.1; no longer R38.2, R39.1
- net N$74: now also R41.1; no longer R40.1
- net N$75: now also R74.1, R82.1, R86.1; no longer R73.1, R81.1, R85.1
- net N$76: now also R86.2; no longer R85.2
- net N$77: now also R100.1; no longer R99.1
- net N$78: now also R101.1; no longer R100.1
- net N$79: now also R75.1, R83.1, R87.1; no longer R74.1, R82.1, R86.1
- net N$80: now also R87.2; no longer R86.2
- net N$81: now also R42.2; no longer R41.2
- net N$82: now also R42.1; no longer R41.1
- net N$83: now also R76.1, R84.1, R88.1; no longer R75.1, R83.1, R87.1
- net N$84: now also R102.2; no longer R101.2
- net N$85: now also R103.2; no longer R102.2
- net N$86: now also R77.1, R85.1, R89.1; no longer R76.1, R84.1, R88.1
- net N$87: now also R88.2; no longer R87.2
- net N$88: now also R89.2; no longer R88.2
- net N$89: now also R90.1; no longer R89.1
- net N$9: now also R20.1, R21.2; no longer R19.1, R20.2
- net N$90: now also R62.1; no longer R61.1
- net N$91: now also R91.1; no longer R90.1
- net N$92: now also R93.1; no longer R92.1
- net N$93: now also R92.1; no longer R91.1
- net N$94: now also R78.1; no longer R77.1
- net N$95: now also R79.1; no longer R78.1
- net N$96: now also R80.1; no longer R79.1
- net N$97: now also R81.1; no longer R80.1
- net N$98: now also R104.2; no longer R103.2
- net N$99: now also R105.2; no longer R104.2
- net OUTPUT1.1: now also R94.2; no longer R93.2
- net OUTPUT1.1_MCU: now also R118.2; no longer R117.2
- net OUTPUT1.2: now also R95.2; no longer R94.2
- net OUTPUT1.2_MCU: now also R119.2; no longer R118.2
- net OUTPUT1.3: now also R96.2; no longer R95.2
- net OUTPUT1.3_MCU: now also R120.2; no longer R119.2
- net OUTPUT1.4: now also R97.2; no longer R96.2
- net OUTPUT1.4_MCU: now also R121.2; no longer R120.2
- net OUTPUT2.1: now also R66.2; no longer R65.2
- net OUTPUT2.1_MCU: now also R90.2; no longer R89.2
- net OUTPUT2.2: now also R67.2; no longer R66.2
- net OUTPUT2.2_MCU: now also R91.2; no longer R90.2
- net OUTPUT2.3: now also R68.2; no longer R67.2
- net OUTPUT2.3_MCU: now also R92.2; no longer R91.2
- net OUTPUT2.4: now also R69.2; no longer R68.2
- net OUTPUT2.4_MCU: now also R93.2; no longer R92.2
- net OUTPUT3.2_MCU: now also R65.2; no longer R64.2
- net USB_D_N: now also R6.2; no longer R5.2
- net USB_D_P: now also R7.2; no longer R6.2
Other:
- moved on the sheet: R10, R100, R101, R102, R103, R104, R105, R106, R107, R108, R109, R11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

Commit message: Replace output resistance and fuse LED
Parts:
- LED3, LED7: MPN OVS-0603 -> OVS-0608; OC_NEWARK 15R2205 -> 15R2208
- R100, R101, R64, R70, R71, R72, R73, R98, R99: value 330 -> 10K; MPN RC0603FR-07330RL -> RC0603FR-0710KL; OC_NEWARK 98K7391 -> 68R0049
- R102, R103, R104, R105, R74, R75, R76, R77: value 100 -> 1K; MPN RC0603FR-13100RL -> RC0603FR-071KL; OC_NEWARK 68R0131 -> 68R0042
- R114, R115, R116, R117, R86, R87, R88, R89: value 1K -> 100; MPN RC0603FR-071KL -> RC0603FR-13100RL; OC_NEWARK 68R0042 -> 68R0131
